Commit message: Reduced height of the robot to the real size

File: ros/src/turtlebot3_description/urdf/turtlebot3_burger_simulation.urdf.xacro (robot description, xacro)
@@ -20,5 +20,5 @@
       <origin xyz="-0.032 0 0.070" rpy="0 0 0"/>
       <geometry>
-        <box size="0.140 0.140 0.143"/>
+        <box size="0.140 0.140 0.083"/>
       </geometry>
     </collision>
